Commit message: Changes for 6 DOF arm

File: panda_description/urdf/panda.urdf (robot description, URDF)
Before this commit: robot panda, 12 links, 11 joints
Links:
- removed link panda_hand
- removed link panda_leftfinger
- removed link panda_link8
- removed link panda_rightfinger
Joints:
- removed joint panda_finger_joint1
- removed joint panda_finger_joint2
- removed joint panda_hand_joint
- removed joint panda_joint8
- joint panda_joint7: axis 0 0 1 -> (none); limit lower=-2.9671 upper=2.9671 effort=12 velocity=2.8710 -> (none); type revolute -> fixed

File: panda_moveit_config/config/panda.urdf.xacro (robot description, xacro)
@@ -7,6 +7,4 @@
     <!-- Import panda ros2_control description -->
     <xacro:include filename="panda.ros2_control.xacro" />
-    <xacro:include filename="panda_hand.ros2_control.xacro" />
     <xacro:panda_ros2_control name="PandaFakeSystem" initial_positions_file="$(arg initial_positions_file)" ros2_control_hardware_type="$(arg ros2_control_hardware_type)"/>
-    <xacro:panda_hand_ros2_control name="PandaHandFakeSystem" ros2_control_hardware_type="$(arg ros2_control_hardware_type)"/>
 </robot>

File: panda_moveit_config/config/panda_arm.xacro (robot description, xacro)
@@ -39,7 +39,4 @@
     </group_state>
     <!--END EFFECTOR: Purpose: Represent information about an end effector.-->
-    <!--VIRTUAL JOINT: Purpose: this element defines a virtual joint between a robot link and an external frame of reference (considered fixed with respect to the robot)-->
-    <virtual_joint name="virtual_joint" type="floating" parent_frame="world" child_link="panda_link0" />
-    <!--DISABLE COLLISIONS: By default it is assumed that any link of the robot could potentially come into collision with any other link in the robot. This tag disables collision checking between a specified pair of links. -->
     <disable_collisions link1="panda_link0" link2="panda_link1" reason="Adjacent" />
     <disable_collisions link1="panda_link0" link2="panda_link2" reason="Never" />
@@ -61,4 +58,5 @@
     <disable_collisions link1="panda_link5" link2="panda_link6" reason="Adjacent" />
     <disable_collisions link1="panda_link6" link2="panda_link7" reason="Adjacent" />
+    <disable_collisions link1="panda_link5" link2="panda_link7" reason="Never" />
   </xacro:macro>
 </robot>

Commit message: Cleaned up URDF

File: panda_description/urdf/panda.urdf (robot description, URDF)
Before this commit: robot panda, 8 links, 7 joints
Links:
- added link ee_base_link
- added link end_effector_link, mass 0.5; collision mesh filename=package://moveit_resources_panda_description/meshes/collisi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; visual mesh filename=package://moveit_resources_panda_description/meshes/visual/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
- added link sliding_link, mass 0.05; collision mesh filename=package://moveit_resources_panda_description/meshes/collisi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; visual mesh filename=package://moveit_resources_panda_description/meshes/visual/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
- added link tip_link
- link panda_link0: mass None -> 2.92
- link panda_link1: mass None -> 2.74
- link panda_link2: mass None -> 2.74
- link panda_link3: mass None -> 2.38
- link panda_link4: mass None -> 2.38
- link panda_link5: mass None -> 2.74
- link panda_link6: mass None -> 1.55
- link panda_link7: mass None -> 0.54
Joints:
- added joint ee_base_link_joint: type fixed, parent tip_link, child ee_base_link, origin xyz=0 0 0 rpy=0 0 0
- added joint ee_connector_joint: type revolute, parent ee_base_link, child end_effector_link, origin xyz=0 0 0 rpy=0 0 0, limit lower=-3.1414 upper=3.1415 effort=12 velocity=2.6100
- added joint slider_joint: type prismatic, parent end_effector_link, child sliding_link, origin xyz=0.14 0.06 -0.003 rpy=0 0 0, axis 1 0 0, limit lower=0 upper=0.1 effort=20.0 velocity=0.5
- added joint tip_joint: type fixed, parent panda_link7, child tip_link, origin xyz=0 0 0.103 rpy=0 -1.57079632679 0
- joint panda_joint5: limit lower=-2.9671 upper=2.9671 effort=12 velocity=2.8710 -> lower=-3.13 upper=3.13 effort=12 velocity=2.8710

File: panda_moveit_config/config/panda.ros2_control.xacro (robot description, xacro)
@@ -68,13 +68,4 @@
                 </state_interface>
             </joint>
-            <joint name="panda_joint7">
-                <command_interface name="position"/>
-                <state_interface name="position">
-                  <param name="initial_value">${initial_positions['panda_joint7']}</param>
-                </state_interface>
-                <state_interface name="velocity">
-                  <param name="initial_value">0.0</param>
-                </state_interface>
-            </joint>
         </ros2_control>
     </xacro:macro>

File: panda_moveit_config/config/panda.urdf.xacro (robot description, xacro)
@@ -7,4 +7,6 @@
     <!-- Import panda ros2_control description -->
     <xacro:include filename="panda.ros2_control.xacro" />
+    <xacro:include filename="panda_hand.ros2_control.xacro" />
     <xacro:panda_ros2_control name="PandaFakeSystem" initial_positions_file="$(arg initial_positions_file)" ros2_control_hardware_type="$(arg ros2_control_hardware_type)"/>
+    <xacro:panda_hand_ros2_control name="PandaHandFakeSystem" initial_positions_file="$(arg initial_positions_file)"  ros2_control_hardware_type="$(arg ros2_control_hardware_type)"/>
 </robot>

File: panda_moveit_config/config/panda_hand.ros2_control.xacro (robot description, xacro)
@@ -1,5 +1,6 @@
 <?xml version="1.0"?>
 <robot xmlns:xacro="http://www.ros.org/wiki/xacro">
-    <xacro:macro name="panda_hand_ros2_control" params="name ros2_control_hardware_type">
+    <xacro:macro name="panda_hand_ros2_control" params="name initial_positions_file ros2_control_hardware_type">
+        <xacro:property name="initial_positions" value="${xacro.load_yaml(initial_positions_file)['initial_positions']}"/>
         <ros2_control name="${name}" type="system">
             <hardware>
@@ -9,26 +10,24 @@
                 <xacro:if value="${ros2_control_hardware_type == 'isaac'}">
                     <plugin>topic_based_ros2_control/TopicBasedSystem</plugin>
-                    <param name="joint_commands_topic">/isaac_joint_commands</param>
+                    <param name="joint_commands_topic">/isaac_joint_commands_ee</param>
                     <param name="joint_states_topic">/isaac_joint_states</param>
                 </xacro:if>
             </hardware>
-            <joint name="panda_finger_joint1">
-                <command_interface name="position" />
+            <joint name="ee_connector_joint">
+                <command_interface name="position"/>
                 <state_interface name="position">
+                  <param name="initial_value">${initial_positions['ee_connector_joint']}</param>
+                </state_interface>
+                <state_interface name="velocity">
                   <param name="initial_value">0.0</param>
                 </state_interface>
-                <state_interface name="velocity">
-                    <param name="initial_value">0.0</param>
-                </state_interface>
             </joint>
-            <joint name="panda_finger_joint2">
-                <param name="mimic">panda_finger_joint1</param>
-                <param name="multiplier">1</param>
-                <command_interface name="position" />
+            <joint name="slider_joint">
+                <command_interface name="position"/>
                 <state_interface name="position">
-                  <param name="initial_value">0.0</param>
+                  <param name="initial_value">${initial_positions['slider_joint']}</param>
                 </state_interface>
                 <state_interface name="velocity">
-                    <param name="initial_value">0.0</param>
+                  <param name="initial_value">0.0</param>
                 </state_interface>
             </joint>

Commit message: Adjust joints to have full revolution

File: panda_description/urdf/panda.urdf (robot description, URDF)
Before this commit: robot panda, 13 links, 12 joints
Links:
- removed link dummy
Joints:
- removed joint dummy_joint
- joint panda_joint1: limit lower=-2.9671 upper=2.9671 effort=87 velocity=2.3925 -> lower=-6.2831853 upper=6.2831853 effort=87 velocity=2.3925
- joint panda_joint5: limit lower=-3.13 upper=3.13 effort=12 velocity=2.8710 -> lower=-6.2831853 upper=6.2831853 effort=12 velocity=2.8710
